Commit message: first attempt for ubuntu 24.04 and ros2 jazzy

File: src/mybots_description/urdf/mybots_gazebo.xacro (robot description, xacro)
@@ -1,19 +1,4 @@
 <?xml version="1.0"?>
 <robot name="mybots" xmlns:xacro="http://ros.org/wiki/xacro">
-  <!-- Move this one to ros2 control -->
-  <transmission name="wheel_right_transmission">
-    <plugin>transmission_interface/SimpleTransmission</plugin>
-    <actuator name="wheel_right_motor" role="actuator_right"/>
-    <joint name="wheel_right_joint"    role="joint_right">
-      <mechanical_reduction>1.0</mechanical_reduction>
-    </joint>
-  </transmission>
-  <transmission name="wheel_left_transmission">
-    <plugin>transmission_interface/SimpleTransmission</plugin>
-    <actuator name="wheel_left_motor" role="actuator_left"/>
-    <joint name="wheel_left_joint"    role="joint_left">
-      <mechanical_reduction>1.0</mechanical_reduction>
-    </joint>
-  </transmission>
   <!-- Wheels -->
   <gazebo reference="wheel_left_link">
@@ -61,12 +46,4 @@
   <gazebo reference="laser_link">
     <material>Gazebo/FlatBlack</material>
-  </gazebo>
-  <!-- ROS 2 Control -->
-  <gazebo>
-    <plugin filename="libgazebo_ros2_control.so" name="gazebo_ros2_control">
-      <robot_param>robot_description</robot_param>
-      <robot_param_node>robot_state_publisher</robot_param_node>
-      <parameters>$(find mybots_controller)/config/mybots_controllers.yaml</parameters>
-    </plugin>
   </gazebo>
   <!-- IMU -->
@@ -117,14 +94,13 @@
           </linear_acceleration>
         </imu>
-        <plugin name="imu" filename="libgazebo_ros_imu_sensor.so"/>
     </sensor>
   </gazebo>
-  <!-- 2D Laser Sensor -->
-  <gazebo reference="laser_link">
-    <sensor name="lidar" type="ray">
+   <!-- 2D Laser Sensor -->
+   <gazebo reference="laser_link">
+    <sensor name="lidar" type="gpu_lidar">
       <always_on>true</always_on>
       <visualize>true</visualize>
       <update_rate>5</update_rate>
-      <ray>
+      <lidar>
         <scan>
           <horizontal>
@@ -145,12 +121,7 @@
           <stddev>0.01</stddev>
         </noise>
-      </ray>
-      <plugin name="scan" filename="libgazebo_ros_ray_sensor.so">
-        <ros>
-          <remapping>~/out:=scan</remapping>
-        </ros>
-        <output_type>sensor_msgs/LaserScan</output_type>
-        <frame_name>laser_link</frame_name>
-      </plugin>
+      </lidar>
+       <topic>scan</topic>
+       <gz_frame_id>laser_link</gz_frame_id>
     </sensor>
   </gazebo>

File: src/mybots_description/urdf/mybots_ros2_control.xacro (robot description, xacro)
@@ -5,5 +5,5 @@
         <xacro:if value="$(arg is_sim)">
             <hardware>
-                <plugin>gazebo_ros2_control/GazeboSystem</plugin>
+                <plugin>gz_ros2_control/GazeboSimSystem</plugin>
             </hardware>
         </xacro:if>
@@ -33,4 +33,23 @@
             <state_interface name="velocity" />
         </joint>
+        <transmission name="wheel_right_transmission">
+            <plugin>transmission_interface/SimpleTransmission</plugin>
+            <actuator name="wheel_right_motor" role="actuator_right"/>
+            <joint name="wheel_right_joint"    role="joint_right">
+            <mechanical_reduction>1.0</mechanical_reduction>
+            </joint>
+        </transmission>
+        <transmission name="wheel_left_transmission">
+            <plugin>transmission_interface/SimpleTransmission</plugin>
+            <actuator name="wheel_left_motor" role="actuator_left"/>
+            <joint name="wheel_left_joint"    role="joint_left">
+            <mechanical_reduction>1.0</mechanical_reduction>
+            </joint>
+        </transmission>
     </ros2_control>
+    <gazebo>
+        <plugin name="gz_ros2_control::GazeboSimROS2ControlPlugin" filename="libgz_ros2_control-system.so">
+            <parameters>$(find mybots_controller)/config/mybots_controllers.yaml</parameters>
+        </plugin>
+    </gazebo>
 </robot>

File: src/mybots_description/urdf/smallbot.urdf.xacro (robot description, xacro)
@@ -1,6 +1,4 @@
 <?xml version="1.0"?>
 <robot name="mybots" xmlns:xacro="http://ros.org/wiki/xacro">
-  <!-- Start GZ or Ignition depending on ROS 2 Version -->
-  <xacro:arg name="is_ignition" default="true"/>
   <!-- Load Simulated or Real Hardware Interfaces -->
   <xacro:arg name="is_sim" default="true"/>

Commit message: xacro revisit but has errors

File: src/mybots_description/urdf/mybots_gazebo.xacro (robot description, xacro)
@@ -47,4 +47,15 @@
     <material>Gazebo/FlatBlack</material>
   </gazebo>
+  <!-- ROS 2 Control -->
+  <gazebo>
+      <plugin name="gz_ros2_control::GazeboSimROS2ControlPlugin" filename="libgz_ros2_control-system.so">
+        <parameters>$(find mybots_controller)/config/mybots_controllers.yaml</parameters>
+      </plugin>
+      <plugin filename="gz-sim-imu-system" name="gz::sim::systems::Imu">
+      </plugin>
+      <plugin filename="gz-sim-sensors-system" name="gz::sim::systems::Sensors">
+        <render_engine>ogre2</render_engine>
+      </plugin>
+  </gazebo>
   <!-- IMU -->
   <gazebo reference="imu_link">
@@ -52,4 +63,6 @@
         <always_on>true</always_on>
         <update_rate>100</update_rate>
+        <gz_frame_id>imu_link</gz_frame_id>
+        <topic>imu</topic>
         <imu>
           <angular_velocity>

File: src/mybots_description/urdf/mybots_ros2_control.xacro (robot description, xacro)
@@ -17,10 +17,4 @@
         </xacro:unless>
         <!-- ros2_control Common Interfaces -->
-        <gazebo>
-            <plugin filename="gz_ros2_control-system" name="gz_ros2_control::GazeboSimROS2ControlPlugin">
-                <parameters>$(find mybots_controller)/config/mybots_controllers.yaml</parameters>
-                <parameters>$(find mybots_controller)/config/config/gaz_ros2_ctl_use_sim.yaml</parameters>
-            </plugin>
-        </gazebo>
         <joint name="wheel_right_joint">
             <command_interface name="velocity">
@@ -39,18 +33,4 @@
             <state_interface name="velocity" />
         </joint>
-        <transmission name="wheel_right_transmission">
-            <plugin>transmission_interface/SimpleTransmission</plugin>
-            <actuator name="wheel_right_motor" role="actuator_right"/>
-            <joint name="wheel_right_joint"    role="joint_right">
-            <mechanical_reduction>1.0</mechanical_reduction>
-            </joint>
-        </transmission>
-        <transmission name="wheel_left_transmission">
-            <plugin>transmission_interface/SimpleTransmission</plugin>
-            <actuator name="wheel_left_motor" role="actuator_left"/>
-            <joint name="wheel_left_joint"    role="joint_left">
-            <mechanical_reduction>1.0</mechanical_reduction>
-            </joint>
-        </transmission>
     </ros2_control>
 </robot>

Commit message: works except safety stop actions

File: src/mybots_description/urdf/mybots_gazebo.xacro (robot description, xacro)
@@ -3,5 +3,4 @@
   <!-- Wheels -->
   <gazebo reference="wheel_left_link">
-    <material>Gazebo/Blue</material>
     <mu1>1000000000000000.0</mu1>
     <mu2>1000000000000000.0</mu2>
@@ -13,5 +12,4 @@
   </gazebo>
   <gazebo reference="wheel_right_link">
-    <material>Gazebo/Blue</material>
     <mu1>1000000000000000.0</mu1>
     <mu2>1000000000000000.0</mu2>
@@ -24,5 +22,4 @@
   <!-- Caster Wheels -->
   <gazebo reference="caster_right_link">
-    <material>Gazebo/FlatBlack</material>
     <mu1>0.1</mu1>
     <mu2>0.1</mu2>
@@ -33,5 +30,4 @@
   </gazebo>
   <gazebo reference="caster_left_link">
-    <material>Gazebo/FlatBlack</material>
     <mu1>0.1</mu1>
     <mu2>0.1</mu2>
@@ -41,10 +37,15 @@
     <maxVel>1.0</maxVel>
   </gazebo>
-  <gazebo reference="base_link">
-    <material>Gazebo/FlatBlack</material>
-  </gazebo>
-  <gazebo reference="laser_link">
-    <material>Gazebo/FlatBlack</material>
-  </gazebo>
+  <!-- ROS 2 Control -->
+  <gazebo>
+    <plugin name="gz_ros2_control::GazeboSimROS2ControlPlugin" filename="libgz_ros2_control-system.so">
+      <parameters>$(find mybots_controller)/config/mybots_controllers.yaml</parameters>
+    </plugin>
+    <plugin filename="gz-sim-imu-system" name="gz::sim::systems::Imu">
+    </plugin>
+    <plugin filename="gz-sim-sensors-system" name="gz::sim::systems::Sensors">
+      <render_engine>ogre2</render_engine>
+    </plugin>
+</gazebo>
   <!-- IMU -->
   <gazebo reference="imu_link">
@@ -52,4 +53,6 @@
         <always_on>true</always_on>
         <update_rate>100</update_rate>
+        <gz_frame_id>imu_link</gz_frame_id>
+        <topic>imu</topic>
         <imu>
           <angular_velocity>
@@ -101,5 +104,7 @@
       <always_on>true</always_on>
       <visualize>true</visualize>
+      <topic>scan</topic>
       <update_rate>5</update_rate>
+      <gz_frame_id>laser_link</gz_frame_id>
       <lidar>
         <scan>
@@ -122,6 +127,4 @@
         </noise>
       </lidar>
-       <topic>scan</topic>
-       <gz_frame_id>laser_link</gz_frame_id>
     </sensor>
   </gazebo>

File: src/mybots_description/urdf/mybots_ros2_control.xacro (robot description, xacro)
@@ -33,23 +33,4 @@
             <state_interface name="velocity" />
         </joint>
-        <transmission name="wheel_right_transmission">
-            <plugin>transmission_interface/SimpleTransmission</plugin>
-            <actuator name="wheel_right_motor" role="actuator_right"/>
-            <joint name="wheel_right_joint"    role="joint_right">
-            <mechanical_reduction>1.0</mechanical_reduction>
-            </joint>
-        </transmission>
-        <transmission name="wheel_left_transmission">
-            <plugin>transmission_interface/SimpleTransmission</plugin>
-            <actuator name="wheel_left_motor" role="actuator_left"/>
-            <joint name="wheel_left_joint"    role="joint_left">
-            <mechanical_reduction>1.0</mechanical_reduction>
-            </joint>
-        </transmission>
     </ros2_control>
-    <gazebo>
-        <plugin name="gz_ros2_control::GazeboSimROS2ControlPlugin" filename="libgz_ros2_control-system.so">
-            <parameters>$(find mybots_controller)/config/mybots_controllers.yaml</parameters>
-        </plugin>
-    </gazebo>
 </robot>
