Commit message: test of urdf file: to find stl

File: src/mybots_description/urdf/smallbot_physical.urdf.xacro (robot description, xacro)
@@ -25,5 +25,5 @@
       <origin xyz="0 0 0" rpy="0 0 0" />
       <geometry>
-        <mesh filename="package://mybots_description/meshes/smallbot_base_link.stl" />
+        <mesh filename="file://$(find mybots_description)/meshes/smallbot_base_link.stl" />
       </geometry>
       <material name="dark_grey"/>

Commit message: changed all stl finds in urdf

File: src/mybots_description/urdf/smallbot_physical.urdf.xacro (robot description, xacro)
@@ -32,5 +32,5 @@
       <origin xyz="0 0 0" rpy="0 0 0" />
       <geometry>
-        <mesh filename="package://mybots_description/meshes/smallbot_base_link.stl" />
+        <mesh filename="file://$(find mybots_description)/meshes/smallbot_base_link.stl" />
       </geometry>
     </collision>
@@ -52,5 +52,5 @@
       <origin xyz="-0.0 0.014 0.0" rpy="1.57 0 0" />
       <geometry>
-        <mesh filename="package://mybots_description/meshes/smallbot_wheel.stl" />
+        <mesh filename="file://$(find mybots_description)/meshes/smallbot_wheel.stl" />
       </geometry>
       <material name="blue"/>
@@ -81,5 +81,5 @@
       <origin xyz="0 -0.014 0" rpy="-1.57 0 0" />
       <geometry>
-        <mesh filename="package://mybots_description/meshes/smallbot_wheel.stl" />
+        <mesh filename="file://$(find mybots_description)/meshes/smallbot_wheel.stl" />
       </geometry>
       <material name="blue"/>
@@ -109,5 +109,5 @@
       <origin xyz="0 0 0" rpy="0 0 0" />
       <geometry>
-        <mesh filename="package://mybots_description/meshes/smallbot_caster_link.stl" />
+        <mesh filename="file://$(find mybots_description)/meshes/smallbot_caster_link.stl" />
       </geometry>
       <material name="silver"/>
@@ -137,5 +137,5 @@
       <origin xyz="0 0 0" rpy="0 0 0" />
       <geometry>
-        <mesh filename="package://mybots_description/meshes/smallbot_caster_link.stl" />
+        <mesh filename="file://$(find mybots_description)/meshes/smallbot_caster_link.stl" />
       </geometry>
       <material name="silver"/>
@@ -165,5 +165,5 @@
       <origin xyz="0 0 0" rpy="0 0 3.14" />
       <geometry>
-        <mesh filename="package://mybots_description/meshes/imu_link.STL" />
+        <mesh filename="file://$(find mybots_description)/meshes/imu_link.STL" />
       </geometry>
       <material name="blue"/>
@@ -172,5 +172,5 @@
       <origin xyz="0 0 0" rpy="0 0 1.57" />
       <geometry>
-        <mesh filename="package://mybots_description/meshes/imu_link.STL" />
+        <mesh filename="file://$(find mybots_description)/meshes/imu_link.STL" />
       </geometry>
     </collision>
@@ -193,5 +193,5 @@
       <origin xyz="0 0 0" rpy="1.57 0 3.14" />
       <geometry>
-        <mesh filename="package://mybots_description/meshes/lidarA1M8.stl" />
+        <mesh filename="file://$(find mybots_description)/meshes/lidarA1M8.stl" />
       </geometry>
       <material name="black"/>
@@ -200,5 +200,5 @@
       <origin xyz="0 0 0" rpy="0 0 0" />
       <geometry>
-        <mesh filename="package://mybots_description/meshes/lidarA1M8.stl" />
+        <mesh filename="file://$(find mybots_description)/meshes/lidarA1M8.stl" />
       </geometry>
     </collision>

Commit message: changed urdf to file://$

File: src/mybots_description/urdf/smallbot_physical.urdf.xacro (robot description, xacro)
@@ -25,5 +25,5 @@
       <origin xyz="0 0 0" rpy="0 0 0" />
       <geometry>
-        <mesh filename="$(find mybots_description)/meshes/smallbot_base_link.stl" />
+        <mesh filename="file://$(find mybots_description)/meshes/smallbot_base_link.stl" />
       </geometry>
       <material name="dark_grey"/>
@@ -32,5 +32,5 @@
       <origin xyz="0 0 0" rpy="0 0 0" />
       <geometry>
-        <mesh filename="$(find mybots_description)/meshes/smallbot_base_link.stl" />
+        <mesh filename="file://$(find mybots_description)/meshes/smallbot_base_link.stl" />
       </geometry>
     </collision>
@@ -52,5 +52,5 @@
       <origin xyz="-0.0 0.014 0.0" rpy="1.57 0 0" />
       <geometry>
-        <mesh filename="$(find mybots_description)/meshes/smallbot_wheel.stl" />
+        <mesh filename="file://$(find mybots_description)/meshes/smallbot_wheel.stl" />
       </geometry>
       <material name="blue"/>
@@ -81,5 +81,5 @@
       <origin xyz="0 -0.014 0" rpy="-1.57 0 0" />
       <geometry>
-        <mesh filename="$(find mybots_description)/meshes/smallbot_wheel.stl" />
+        <mesh filename="file://$(find mybots_description)/meshes/smallbot_wheel.stl" />
       </geometry>
       <material name="blue"/>
@@ -109,5 +109,5 @@
       <origin xyz="0 0 0" rpy="0 0 0" />
       <geometry>
-        <mesh filename="$(find mybots_description)/meshes/smallbot_caster_link.stl" />
+        <mesh filename="file://$(find mybots_description)/meshes/smallbot_caster_link.stl" />
       </geometry>
       <material name="silver"/>
@@ -137,5 +137,5 @@
       <origin xyz="0 0 0" rpy="0 0 0" />
       <geometry>
-        <mesh filename="$(find mybots_description)/meshes/smallbot_caster_link.stl" />
+        <mesh filename="file://$(find mybots_description)/meshes/smallbot_caster_link.stl" />
       </geometry>
       <material name="silver"/>
@@ -165,5 +165,5 @@
       <origin xyz="0 0 0" rpy="0 0 3.14" />
       <geometry>
-        <mesh filename="$(find mybots_description)/meshes/imu_link.STL" />
+        <mesh filename="file://$(find mybots_description)/meshes/imu_link.STL" />
       </geometry>
       <material name="blue"/>
@@ -172,5 +172,5 @@
       <origin xyz="0 0 0" rpy="0 0 1.57" />
       <geometry>
-        <mesh filename="$(find mybots_description)/meshes/imu_link.STL" />
+        <mesh filename="file://$(find mybots_description)/meshes/imu_link.STL" />
       </geometry>
     </collision>
@@ -193,5 +193,5 @@
       <origin xyz="0 0 0" rpy="1.57 0 3.14" />
       <geometry>
-        <mesh filename="$(find mybots_description)/meshes/lidarA1M8.stl" />
+        <mesh filename="file://$(find mybots_description)/meshes/lidarA1M8.stl" />
       </geometry>
       <material name="black"/>
@@ -200,5 +200,5 @@
       <origin xyz="0 0 0" rpy="0 0 0" />
       <geometry>
-        <mesh filename="$(find mybots_description)/meshes/lidarA1M8.stl" />
+        <mesh filename="file://$(find mybots_description)/meshes/lidarA1M8.stl" />
       </geometry>
     </collision>

Commit message: change imu_joint to continuous

File: src/mybots_description/urdf/smallbot_physical.urdf.xacro (robot description, xacro)
@@ -176,5 +176,5 @@
     </collision>
   </link>
-  <joint name="imu_joint" type="fixed">
+  <joint name="imu_joint" type="continuous">
     <origin xyz="-0.04016 0.049755 0.064953" rpy="3.14 0 -1.57" />
     <parent link="base_link" />

Commit message: more on imu inclusion

File: src/mybots_description/urdf/smallbot_physical.urdf.xacro (robot description, xacro)
@@ -176,5 +176,5 @@
     </collision>
   </link>
-  <joint name="imu_joint" type="continuous">
+  <joint name="imu_joint" type="fixed">
     <origin xyz="-0.04016 0.049755 0.064953" rpy="3.14 0 -1.57" />
     <parent link="base_link" />
