Commit message: clean up urdf files

File: src/mybots_description/urdf/mybots_gazebo_control.xacro (robot description, xacro)
@@ -1,4 +1,10 @@
 <?xml version="1.0"?>
 <robot name="mybots" xmlns:xacro="http://ros.org/wiki/xacro">
+    <!-- ROS 2 Control -->
+    <gazebo>
+      <plugin name="gz_ros2_control::GazeboSimROS2ControlPlugin" filename="libgz_ros2_control-system.so">
+        <parameters>$(find mybots_controller)/config/mybots_controllers.yaml</parameters>
+      </plugin>
+  </gazebo>
   <!-- Wheels -->
   <gazebo reference="wheel_left_link">
@@ -37,15 +43,4 @@
     <maxVel>1.0</maxVel>
   </gazebo>
-  <!-- ROS 2 Control -->
-  <gazebo>
-    <plugin name="gz_ros2_control::GazeboSimROS2ControlPlugin" filename="libgz_ros2_control-system.so">
-      <parameters>$(find mybots_controller)/config/mybots_controllers.yaml</parameters>
-    </plugin>
-    <plugin filename="gz-sim-imu-system" name="gz::sim::systems::Imu">
-    </plugin>
-    <plugin filename="gz-sim-sensors-system" name="gz::sim::systems::Sensors">
-      <render_engine>ogre2</render_engine>
-    </plugin>
-</gazebo>
   <!-- IMU -->
   <gazebo reference="imu_link">

File: src/mybots_description/urdf/smallbot.urdf.xacro (robot description, xacro)
@@ -2,217 +2,12 @@
 <robot name="mybots" xmlns:xacro="http://ros.org/wiki/xacro">
   <!-- Load Simulated or Real Hardware Interfaces -->
-  <xacro:arg name="is_sim" default="true"/>
-  <!-- Include Gazebo Parameters -->
-  <xacro:include filename="$(find mybots_description)/urdf/mybots_gazebo.xacro" />
-  <!-- Include ros2_control Plugins -->
+   <xacro:arg name="is_sim" default="true"/>
+  <!-- Include physical aspects of the robot, includes LIDAR and IMU -->
+  <xacro:include filename="$(find mybots_description)/urdf/smallbot_physical.urdf.xacro" />
+  <!-- Include ros2 control Parameters for both SIM and REAL robots-->
   <xacro:include filename="$(find mybots_description)/urdf/mybots_ros2_control.xacro" />
-  <link name="base_footprint"/>
-  <link name="base_link">
-    <inertial>
-      <origin xyz="-0.070489 -0.000718 0.040699" rpy="0.0 0.0 0.0" />
-      <mass value="1.409448"/>
-      <inertia ixx="0.011114" ixy="0.000188" ixz="-0.005821"
-               iyy="0.017229" iyz="0.000127"
-               izz="0.019734" />
-    </inertial>
-    <visual>
-      <origin xyz="0 0 0" rpy="0 0 0" />
-      <geometry>
-        <mesh filename="package://mybots_description/meshes/smallbot_base_link.stl" />
-      </geometry>
-      <material name="dark_grey"/>
-    </visual>
-    <collision>
-      <origin xyz="0 0 0" rpy="0 0 0" />
-      <geometry>
-        <mesh filename="package://mybots_description/meshes/smallbot_base_link.stl" />
-      </geometry>
-    </collision>
-  </link>
-  <joint name="base_joint" type="fixed">
-    <parent link="base_footprint"/>
-    <child link="base_link" />
-    <origin xyz="0 0 0.033" rpy="0 0 0"/>
-  </joint>
-  <link name="wheel_right_link">
-    <inertial>
-      <origin xyz="0 -0.014 0" rpy="0 0 0" />
-      <mass value="0.0530086090966721" />
-      <inertia ixx="1.88176298336665E-05" ixy="-4.8444933029987E-10" ixz="1.88163708851143E-08"
-               iyy="3.11510738647764E-05" iyz="-6.93560663069607E-11"
-               izz="1.8801969558182E-05" />
-    </inertial>
-    <visual>
-      <origin xyz="-0.0 0.014 0.0" rpy="1.57 0 0" />
-      <geometry>
-        <mesh filename="package://mybots_description/meshes/smallbot_wheel.stl" />
-      </geometry>
-      <material name="blue"/>
-    </visual>
-    <collision>
-      <origin xyz="0 -0.015 0" rpy="1.57 0 0" />
-      <geometry>
-        <sphere radius="0.033"/>
-      </geometry>
-    </collision>
-  </link>
-  <joint name="wheel_right_joint" type="continuous">
-    <origin xyz="0 -0.141 0" rpy="0 0 0" />
-    <parent link="base_link" />
-    <child link="wheel_right_link" />
-    <axis xyz="0 1 0" />
-  </joint>
-  <link
-    name="wheel_left_link">
-    <inertial>
-      <origin xyz="0 -0.014 0" rpy="0 0 0" />
-      <mass value="0.0530086043217644" />
-      <inertia ixx="1.8792911368909E-05"  ixy="3.31256392204584E-10" ixz="-1.14082001662767E-08"
-               iyy="3.11510738759073E-05" iyz="-3.60499245082192E-10"
-               izz="1.88266886146847E-05" />
-    </inertial>
-    <visual>
-      <origin xyz="0 -0.014 0" rpy="-1.57 0 0" />
-      <geometry>
-        <mesh filename="package://mybots_description/meshes/smallbot_wheel.stl" />
-      </geometry>
-      <material name="blue"/>
-    </visual>
-    <collision>
-      <origin xyz="0 -0.014 0" rpy="-1.57 0 0" />
-      <geometry>
-        <sphere radius="0.033"/>
-      </geometry>
-    </collision>
-  </link>
-  <joint name="wheel_left_joint" type="continuous">
-    <origin xyz="0 0.141 0" rpy="0 0 0" />
-    <parent link="base_link" />
-    <child link="wheel_left_link" />
-    <axis xyz="0 1 0" />
-  </joint>
-  <link name="caster_right_link">
-    <inertial>
-      <origin xyz=".000112 -0.0155 -.00818" rpy="0 0 0" />
-      <mass value="0.027976" />
-      <inertia ixx="0.000019" ixy="0" ixz="0"
-               iyy="0.000007"  iyz="0.000006"
-               izz="0.000014" />
-    </inertial>
-    <visual>
-      <origin xyz="0 0 0" rpy="0 0 0" />
-      <geometry>
-        <mesh filename="package://mybots_description/meshes/smallbot_caster_link.stl" />
-      </geometry>
-      <material name="silver"/>
-    </visual>
-    <collision>
-      <origin xyz="0 0 0" rpy="0 0 0" />
-      <geometry>
-        <sphere radius="0.051"/>
-      </geometry>
-    </collision>
-  </link>
-  <joint name="caster_right_joint" type="fixed">
-    <origin xyz="-0.137 -0.095 .0133" rpy="1.57 0 1.57" />
-    <parent link="base_link" />
-    <child link="caster_right_link" />
-    <axis xyz="0 0 0" />
-  </joint>
-  <link name="caster_left_link">
-    <inertial>
-      <origin xyz=".000112 -0.0155 -.00818" rpy="0 0 0" />
-      <mass value="0.027976" />
-      <inertia ixx="0.000019" ixy="0" ixz="0"
-               iyy="0.000007"  iyz="0.000006"
-               izz="0.000014" />
-    </inertial>
-    <visual>
-      <origin xyz="0 0 0" rpy="0 0 0" />
-      <geometry>
-        <mesh filename="package://mybots_description/meshes/smallbot_caster_link.stl" />
-      </geometry>
-      <material name="silver"/>
-    </visual>
-    <collision>
-      <origin xyz="0 0 0" rpy="0 0 0" />
-      <geometry>
-        <sphere radius="0.051"/>
-      </geometry>
-    </collision>
-  </link>
-  <joint name="caster_left_joint" type="fixed">
-    <origin xyz="-0.137 0.095 0.0133" rpy="1.57 0 1.57" />
-    <parent link="base_link" />
-    <child link="caster_left_link" />
-    <axis xyz="0 0 0" />
-  </joint>
-  <link name="imu_link">
-    <inertial>
-      <origin xyz="-0.00552433659106688 0.000168210391520346 0.000514000497342681" rpy="0 0 0" />
-      <mass value="0.000528415362211671" />
-      <inertia ixx="1.46176048428261E-08" ixy="1.40015117949421E-10" ixz="-1.99633872937403E-12"
-               iyy="8.59662482954888E-09" iyz="7.52375112767959E-12"
-               izz="2.30279421279312E-08" />
-    </inertial>
-    <visual>
-      <origin xyz="0 0 0" rpy="0 0 3.14" />
-      <geometry>
-        <mesh filename="package://mybots_description/meshes/imu_link.STL" />
-      </geometry>
-      <material name="blue"/>
-    </visual>
-    <collision>
-      <origin xyz="0 0 0" rpy="0 0 1.57" />
-      <geometry>
-        <mesh filename="package://mybots_description/meshes/imu_link.STL" />
-      </geometry>
-    </collision>
-  </link>
-  <joint name="imu_joint" type="fixed">
-    <origin xyz="-0.04016 0.049755 0.064953" rpy="3.14 0 -1.57" />
-    <parent link="base_link" />
-    <child link="imu_link" />
-    <axis xyz="0 0 0" />
-  </joint>
-  <link name="laser_link">
-    <inertial>
-      <origin xyz="0.005399 -0.010876 0.002517" rpy="0 0 0" />
-      <mass value="0.07308" />
-      <inertia ixx="0.000039" ixy="-0.000011" ixz="0.000003"
-               iyy="0.000063" iyz="-0.000005"
-               izz="0.000057" />
-    </inertial>
-    <visual>
-      <origin xyz="0 0 0" rpy="1.57 0 3.14" />
-      <geometry>
-        <mesh filename="package://mybots_description/meshes/lidarA1M8.stl" />
-      </geometry>
-      <material name="black"/>
-    </visual>
-    <collision>
-      <origin xyz="0 0 0" rpy="0 0 0" />
-      <geometry>
-        <mesh filename="package://mybots_description/meshes/lidarA1M8.stl" />
-      </geometry>
-    </collision>
-  </link>
-  <joint name="laser_joint" type="fixed">
-    <origin xyz="-0.013456 0.000513 0.140452" rpy="0 0 3.14" />
-    <parent link="base_link" />
-    <child link="laser_link" />
-    <axis xyz="0 0 0" />
-  </joint>
-  <material name="blue">
-    <color rgba="0 0 1 1"/>
-  </material>
-  <material name="black">
-    <color rgba="0 0 0 1"/>
-  </material>
-  <material name="silver">
-    <color rgba="0.79 0.82 0.93 1"/>
-  </material>
-  <material name="dark_grey">
-    <color rgba="0.3 0.3 0.3 1"/>
-  </material>
+  <!-- Include gazebo Plugins for SIM only -->
+  <xacro:if value="$(arg is_sim)">
+      <xacro:include filename="$(find mybots_description)/urdf/mybots_gazebo_control.xacro" />
+  </xacro:if>
 </robot>

File: src/mybots_description/urdf/smallbot_physical.urdf.xacro (robot description, xacro)
@@ -1,29 +1,36 @@
 <?xml version="1.0"?>
 <robot name="mybots" xmlns:xacro="http://ros.org/wiki/xacro">
-  <!-- Load Simulated or Real Hardware Interfaces -->
-  <xacro:arg name="is_sim" default="true"/>
-  <!-- Include Gazebo Parameters -->
-  <xacro:include filename="$(find mybots_description)/urdf/mybots_gazebo.xacro" />
-  <!-- Include ros2_control Plugins -->
-  <xacro:include filename="$(find mybots_description)/urdf/mybots_ros2_control.xacro" />
+  <material name="blue">
+    <color rgba="0 0 1 1"/>
+  </material>
+  <material name="black">
+    <color rgba="0 0 0 1"/>
+  </material>
+  <material name="silver">
+    <color rgba="0.79 0.82 0.93 1"/>
+  </material>
+  <material name="dark_grey">
+    <color rgba="0.3 0.3 0.3 1"/>
+  </material>
   <link name="base_footprint"/>
   <link name="base_link">
     <inertial>
-      <origin xyz="0 0 0.04" rpy="0.0 0.25 0.3" />
-      <mass value="1.0"/>
-      <inertia ixx="2.2124416e-02" ixy="-1.2294101e-04" ixz="3.4938785e-04"
-               iyy="2.1193702e-02" iyz="-5.0120904e-05"
-               izz="2.0064271e-02" />
-    </inertial>
-    <visual>
-      <origin xyz="0 0 0" rpy="0 0 0" />
-      <geometry>
-        <mesh filename="package://mybots_description/meshes/base_link.STL" />
-      </geometry>
-    </visual>
-    <collision>
-      <origin xyz="0 0 0" rpy="0 0 0" />
-      <geometry>
-        <mesh filename="package://mybots_description/meshes/base_link.STL" />
+      <origin xyz="-0.070489 -0.000718 0.040699" rpy="0.0 0.0 0.0" />
+      <mass value="1.409448"/>
+      <inertia ixx="0.011114" ixy="0.000188" ixz="-0.005821"
+               iyy="0.017229" iyz="0.000127"
+               izz="0.019734" />
+    </inertial>
+    <visual>
+      <origin xyz="0 0 0" rpy="0 0 0" />
+      <geometry>
+        <mesh filename="package://mybots_description/meshes/smallbot_base_link.stl" />
+      </geometry>
+      <material name="dark_grey"/>
+    </visual>
+    <collision>
+      <origin xyz="0 0 0" rpy="0 0 0" />
+      <geometry>
+        <mesh filename="package://mybots_description/meshes/smallbot_base_link.stl" />
       </geometry>
     </collision>
@@ -37,5 +44,5 @@
     <inertial>
       <origin xyz="0 -0.014 0" rpy="0 0 0" />
-      <mass value="1.0" />
+      <mass value="0.0530086090966721" />
       <inertia ixx="1.88176298336665E-05" ixy="-4.8444933029987E-10" ixz="1.88163708851143E-08"
                iyy="3.11510738647764E-05" iyz="-6.93560663069607E-11"
@@ -43,8 +50,9 @@
     </inertial>
     <visual>
-      <origin xyz="0 0 0" rpy="1.57 0 0" />
-      <geometry>
-        <mesh filename="package://mybots_description/meshes/wheel_right_link.STL" />
-      </geometry>
+      <origin xyz="-0.0 0.014 0.0" rpy="1.57 0 0" />
+      <geometry>
+        <mesh filename="package://mybots_description/meshes/smallbot_wheel.stl" />
+      </geometry>
+      <material name="blue"/>
     </visual>
     <collision>
@@ -64,6 +72,6 @@
     name="wheel_left_link">
     <inertial>
-      <origin xyz="0 0.014 0" rpy="0 0 0" />
-      <mass value="1.0" />
+      <origin xyz="0 -0.014 0" rpy="0 0 0" />
+      <mass value="0.0530086043217644" />
       <inertia ixx="1.8792911368909E-05"  ixy="3.31256392204584E-10" ixz="-1.14082001662767E-08"
                iyy="3.11510738759073E-05" iyz="-3.60499245082192E-10"
@@ -71,11 +79,12 @@
     </inertial>
     <visual>
-      <origin xyz="0 0 0" rpy="-1.57 0 0" />
-      <geometry>
-        <mesh filename="package://mybots_description/meshes/wheel_left_link.STL" />
-      </geometry>
-    </visual>
-    <collision>
-      <origin xyz="0 0.015 0" rpy="-1.57 0 0" />
+      <origin xyz="0 -0.014 0" rpy="-1.57 0 0" />
+      <geometry>
+        <mesh filename="package://mybots_description/meshes/smallbot_wheel.stl" />
+      </geometry>
+      <material name="blue"/>
+    </visual>
+    <collision>
+      <origin xyz="0 -0.014 0" rpy="-1.57 0 0" />
       <geometry>
         <sphere radius="0.033"/>
@@ -89,56 +98,58 @@
     <axis xyz="0 1 0" />
   </joint>
+  <link name="caster_right_link">
+    <inertial>
+      <origin xyz=".000112 -0.0155 -.00818" rpy="0 0 0" />
+      <mass value="0.027976" />
+      <inertia ixx="0.000019" ixy="0" ixz="0"
+               iyy="0.000007"  iyz="0.000006"
+               izz="0.000014" />
+    </inertial>
+    <visual>
+      <origin xyz="0 0 0" rpy="0 0 0" />
+      <geometry>
+        <mesh filename="package://mybots_description/meshes/smallbot_caster_link.stl" />
+      </geometry>
+      <material name="silver"/>
+    </visual>
+    <collision>
+      <origin xyz="0 0 0" rpy="0 0 0" />
+      <geometry>
+        <sphere radius="0.051"/>
+      </geometry>
+    </collision>
+  </link>
+  <joint name="caster_right_joint" type="fixed">
+    <origin xyz="-0.137 -0.095 .0133" rpy="1.57 0 1.57" />
+    <parent link="base_link" />
+    <child link="caster_right_link" />
+    <axis xyz="0 0 0" />
+  </joint>
   <link name="caster_left_link">
     <inertial>
-      <origin xyz="3.89968128948481E-07 2.40073004698083E-07 0.00219173397061506" rpy="0 0 0" />
-      <mass value="1.44379265037903E-06" />
-      <inertia ixx="7.23075276010246E-11" ixy="-6.10956883467859E-16" ixz="2.22849693525031E-15"
-               iyy="3.8713793085917E-11"  iyz="2.93909858781952E-15"
-               izz="1.00967486676306E-10" />
-    </inertial>
-    <visual>
-      <origin xyz="0 0 0" rpy="0 0 0" />
-      <geometry>
-        <mesh filename="package://mybots_description/meshes/caster_front_link.STL" />
-      </geometry>
-    </visual>
-    <collision>
-      <origin xyz="0 0 0" rpy="0 0 0" />
-      <geometry>
-        <sphere radius="0.005"/>
+      <origin xyz=".000112 -0.0155 -.00818" rpy="0 0 0" />
+      <mass value="0.027976" />
+      <inertia ixx="0.000019" ixy="0" ixz="0"
+               iyy="0.000007"  iyz="0.000006"
+               izz="0.000014" />
+    </inertial>
+    <visual>
+      <origin xyz="0 0 0" rpy="0 0 0" />
+      <geometry>
+        <mesh filename="package://mybots_description/meshes/smallbot_caster_link.stl" />
+      </geometry>
+      <material name="silver"/>
+    </visual>
+    <collision>
+      <origin xyz="0 0 0" rpy="0 0 0" />
+      <geometry>
+        <sphere radius="0.051"/>
       </geometry>
     </collision>
   </link>
   <joint name="caster_left_joint" type="fixed">
-    <origin xyz="0.04755 0 -0.0275" rpy="0 0 0" />
+    <origin xyz="-0.137 0.095 0.0133" rpy="1.57 0 1.57" />
     <parent link="base_link" />
     <child link="caster_left_link" />
-    <axis xyz="0 0 0" />
-  </joint>
-  <link name="caster_right_link">
-    <inertial>
-      <origin xyz="3.8996812895542E-07 2.40073004698083E-07 0.00219173397061509" rpy="0 0 0" />
-      <mass value="1.44379265037902E-06" />
-      <inertia ixx="7.23075276010246E-11" ixy="-6.10956872363424E-16" ixz="2.22849693527207E-15"
-               iyy="3.87137930859167E-11" iyz="2.939098587861E-15"
-               izz="1.00967486676306E-10" />
-    </inertial>
-    <visual>
-      <origin xyz="0 0 0" rpy="0 0 0" />
-      <geometry>
-        <mesh filename="package://mybots_description/meshes/caster_rear_link.STL" />
-      </geometry>
-    </visual>
-    <collision>
-      <origin xyz="0 0 0" rpy="0 0 0" />
-      <geometry>
-        <sphere radius="0.005"/>
-      </geometry>
-    </collision>
-  </link>
-  <joint name="caster_right_joint" type="fixed">
-    <origin xyz="-0.04755 0 -0.0275" rpy="0 0 0" />
-    <parent link="base_link" />
-    <child link="caster_right_link" />
     <axis xyz="0 0 0" />
   </joint>
@@ -152,11 +163,12 @@
     </inertial>
     <visual>
-      <origin xyz="0 0 0" rpy="0 0 0" />
+      <origin xyz="0 0 0" rpy="0 0 3.14" />
       <geometry>
         <mesh filename="package://mybots_description/meshes/imu_link.STL" />
       </geometry>
-    </visual>
-    <collision>
-      <origin xyz="0 0 0" rpy="0 0 0" />
+      <material name="blue"/>
+    </visual>
+    <collision>
+      <origin xyz="0 0 0" rpy="0 0 1.57" />
       <geometry>
         <mesh filename="package://mybots_description/meshes/imu_link.STL" />
@@ -165,5 +177,5 @@
   </link>
   <joint name="imu_joint" type="fixed">
-    <origin xyz="0 0 0.0698986241758014" rpy="0 0 0" />
+    <origin xyz="-0.04016 0.049755 0.064953" rpy="3.14 0 -1.57" />
     <parent link="base_link" />
     <child link="imu_link" />
@@ -172,25 +184,26 @@
   <link name="laser_link">
     <inertial>
-      <origin xyz="-0.011945780406062 -0.000381929217680526 -0.0170649378129477" rpy="0 0 0" />
-      <mass value="0.073084435549317" />
-      <inertia ixx="1.96074931730795E-05" ixy="-3.62091076640009E-07" ixz="4.28230084046735E-07"
-               iyy="2.40983835136327E-05" iyz="1.50180909250652E-08"
-               izz="4.14184164228595E-05" />
-    </inertial>
-    <visual>
-      <origin xyz="0 0 0" rpy="0 0 0" />
-      <geometry>
-        <mesh filename="package://mybots_description/meshes/laser_link.STL" />
-      </geometry>
-    </visual>
-    <collision>
-      <origin xyz="0 0 0" rpy="0 0 0" />
-      <geometry>
-        <mesh filename="package://mybots_description/meshes/laser_link.STL" />
+      <origin xyz="0.005399 -0.010876 0.002517" rpy="0 0 0" />
+      <mass value="0.07308" />
+      <inertia ixx="0.000039" ixy="-0.000011" ixz="0.000003"
+               iyy="0.000063" iyz="-0.000005"
+               izz="0.000057" />
+    </inertial>
+    <visual>
+      <origin xyz="0 0 0" rpy="1.57 0 3.14" />
+      <geometry>
+        <mesh filename="package://mybots_description/meshes/lidarA1M8.stl" />
+      </geometry>
+      <material name="black"/>
+    </visual>
+    <collision>
+      <origin xyz="0 0 0" rpy="0 0 0" />
+      <geometry>
+        <mesh filename="package://mybots_description/meshes/lidarA1M8.stl" />
       </geometry>
     </collision>
   </link>
   <joint name="laser_joint" type="fixed">
-    <origin xyz="-0.0050526 -0.0023221 0.1208" rpy="0 0 3.14" />
+    <origin xyz="-0.013456 0.000513 0.140452" rpy="0 0 3.14" />
     <parent link="base_link" />
     <child link="laser_link" />

Commit message: laser_link to laser_frame

File: src/mybots_description/urdf/mybots_gazebo_control.xacro (robot description, xacro)
@@ -95,5 +95,5 @@
   </gazebo>
    <!-- 2D Laser Sensor -->
-   <gazebo reference="laser_link">
+   <gazebo reference="laser_frame">
     <sensor name="lidar" type="gpu_lidar">
       <always_on>true</always_on>
@@ -101,5 +101,5 @@
       <topic>scan</topic>
       <update_rate>5</update_rate>
-      <gz_frame_id>laser_link</gz_frame_id>
+      <gz_frame_id>laser_frame</gz_frame_id>
       <lidar>
         <scan>

File: src/mybots_description/urdf/smallbot_physical.urdf.xacro (robot description, xacro)
@@ -182,5 +182,5 @@
     <axis xyz="0 0 0" />
   </joint>
-  <link name="laser_link">
+  <link name="laser_frame">
     <inertial>
       <origin xyz="0.005399 -0.010876 0.002517" rpy="0 0 0" />
@@ -207,5 +207,5 @@
     <origin xyz="-0.013456 0.000513 0.140452" rpy="0 0 3.14" />
     <parent link="base_link" />
-    <child link="laser_link" />
+    <child link="laser_frame" />
     <axis xyz="0 0 0" />
   </joint>
