Commit message: base left arm manual move & mqtt serial print removed

File: src/mybots_description/urdf/mybots_gazebo_control.xacro (robot description, xacro)
@@ -4,5 +4,5 @@
   <xacro:if value="$(arg is_sim)">
     <gazebo>
-      <plugin name="gz_ros2_control::GazeboSimROS2ControlPlugin" filename="libgz_ros2_control-system.so">
+      <plugin name="gz_ros2_control::GazeboSimROS2ControlPlugin" filename="gz_ros2_control-system">
         <parameters>$(find mybots_controller)/config/mybots_controllers.yaml</parameters>
       </plugin>
@@ -126,3 +126,72 @@
     </sensor>
   </gazebo>
+  <!-- rgb camera -->
+  <gazebo reference="rgb_camera">
+    <sensor name="camera" type="camera">
+      <always_on>true</always_on>
+      <visualize>true</visualize>
+      <topic>/image_raw</topic>
+      <update_rate>30</update_rate>
+      <gz_frame_id>/rgb_camera</gz_frame_id>
+      <camera name="camera">
+        <horizontal_fov>1.21126</horizontal_fov>
+        <vertical_fov>0.71</vertical_fov>
+        <image>
+            <width>2304</width>
+            <height>1296</height>
+            <format>R8G8B8</format>
+        </image>
+        <distortion>
+            <k1>0.0</k1>
+            <k2>0.0</k2>
+            <k3>0.0</k3>
+            <p1>0.0</p1>
+            <p2>0.0</p2>
+            <center>0.5 0.5</center>
+        </distortion>
+      </camera>
+    </sensor>
+  </gazebo>
+    <!-- left arm joints
+  <gazebo reference="joint_1">
+    <mu1>0.1</mu1>
+    <mu2>0.1</mu2>
+    <kp>1000000.0</kp>
+    <kd>100.0</kd>
+    <minDepth>0.001</minDepth>
+    <maxVel>1.0</maxVel>
+  </gazebo>
+  <gazebo reference="joint_2">
+    <mu1>0.1</mu1>
+    <mu2>0.1</mu2>
+    <kp>1000000.0</kp>
+    <kd>100.0</kd>
+    <minDepth>0.001</minDepth>
+    <maxVel>1.0</maxVel>
+  </gazebo>
+  <gazebo reference="joint_3">
+    <mu1>0.1</mu1>
+    <mu2>0.1</mu2>
+    <kp>1000000.0</kp>
+    <kd>100.0</kd>
+    <minDepth>0.001</minDepth>
+    <maxVel>1.0</maxVel>
+  </gazebo>
+  <gazebo reference="joint_4">
+    <mu1>0.1</mu1>
+    <mu2>0.1</mu2>
+    <kp>1000000.0</kp>
+    <kd>100.0</kd>
+    <minDepth>0.001</minDepth>
+    <maxVel>1.0</maxVel>
+  </gazebo>
+  <gazebo reference="joint_1">
+    <mu1>0.1</mu1>
+    <mu2>0.1</mu2>
+    <kp>1000000.0</kp>
+    <kd>100.0</kd>
+    <minDepth>0.001</minDepth>
+    <maxVel>1.0</maxVel>
+  </gazebo>
+  -->
 </robot>

File: src/mybots_description/urdf/mybots_ros2_control.xacro (robot description, xacro)
@@ -33,4 +33,36 @@
             <state_interface name="velocity" />
         </joint>
+        <joint name="joint_1">
+            <command_interface name="position">
+              <param name="min">-1.57</param>
+              <param name="max">1.57</param>
+            </command_interface>
+            <state_interface name="position" />
+        </joint>
+        <joint name="joint_2">
+            <command_interface name="position">
+              <param name="min">-1.57</param>
+              <param name="max">1.57</param>
+            </command_interface>
+            <state_interface name="position" />
+        </joint>
+        <joint name="joint_3">
+            <command_interface name="position">
+              <param name="min">-1.57</param>
+              <param name="max">1.57</param>
+            </command_interface>
+            <state_interface name="position" />
+        </joint>
+        <joint name="joint_4">
+            <command_interface name="position">
+              <param name="min">-1.57</param>
+              <param name="max">0</param>
+            </command_interface>
+            <state_interface name="position" />
+        </joint>
+        <joint name="joint_5">
+            <param name="mimic">joint_4</param>
+            <param name="multiplier">-1</param>
+        </joint>
     </ros2_control>
 </robot>

File: src/mybots_description/urdf/smallbot.urdf.xacro (robot description, xacro)
@@ -4,6 +4,7 @@
    <xacro:arg name="is_sim" default="true"/>
    <xacro:arg name="use_ros2_control" default="true"/>
-  <!-- Include physical aspects of the robot, includes LIDAR and IMU -->
+  <!-- Include physical aspects of the robot, includes add-ons -->
   <xacro:include filename="$(find mybots_description)/urdf/smallbot_physical.urdf.xacro" />
+  <xacro:include filename="$(find mybots_description)/urdf/little_arm.urdf.xacro" />
   <!-- Include ros2 control Parameters for both SIM and REAL robots-->
   <xacro:include filename="$(find mybots_description)/urdf/mybots_ros2_control.xacro" />

File: src/mybots_description/urdf/smallbot_physical.urdf.xacro (robot description, xacro)
@@ -6,4 +6,7 @@
   <material name="black">
     <color rgba="0 0 0 1"/>
+  </material>
+  <material name="white">
+  <color rgba="1 1 1 1"/>
   </material>
   <material name="silver">
