Commit message: working sim with moveIt, Alexa not working

File: src/mybots_description/urdf/little_arm.urdf.xacro (robot description, xacro)
@@ -1,3 +1,3 @@
-<?xml version="1.0"?>
+<?xml version="0.001"?>
 <robot xmlns:xacro="http://www.ros.org/wiki/xacro" name="little_arm">
     <!-- Useful XACRO Variables (Properties) -->
@@ -10,7 +10,7 @@
             <origin xyz="0 0 0" rpy="0 0 0"/>
             <mass value="${mass}" />
-            <inertia ixx="1.0" ixy="0.0" ixz="0.0"
-                     iyy="1.0" iyz="0.0"
-                     izz="1.0" />
+            <inertia ixx="0.001" ixy="0.0" ixz="0.0"
+                     iyy="0.001" iyz="0.0"
+                     izz="0.001" />
         </inertial>
     </xacro:macro>
@@ -18,5 +18,5 @@
     <link name="world"/> -->
     <link name="basement">
-        <xacro:default_inertial mass="1.0"/>
+        <xacro:default_inertial mass="0.028"/>
         <visual>
             <origin rpy="0 0 0" xyz="-0.05 -0.05 0"/>
@@ -34,5 +34,5 @@
     </link>
     <link name="base_plate">
-        <xacro:default_inertial mass="0.1"/>
+        <xacro:default_inertial mass="0.023"/>
         <visual>
             <origin rpy="0 0 0" xyz="-0.039 -0.039 -0.056"/>
@@ -49,5 +49,5 @@
     </link>
     <link name="forward_drive_arm">
-        <xacro:default_inertial mass="0.1"/>
+        <xacro:default_inertial mass="0.009"/>
         <visual>
             <origin rpy=" 0 -${PI / 2} ${PI / 2}" xyz="0.019 0.006 -0.008"/>
@@ -64,5 +64,5 @@
     </link>
     <link name="horizontal_arm">
-        <xacro:default_inertial mass="0.1"/>
+        <xacro:default_inertial mass="0.006"/>
         <visual>
             <origin rpy="${PI / 2} 0 ${PI / 2}" xyz="-0.003 -0.04 -0.006"/>
@@ -79,5 +79,5 @@
     </link>
     <link name="claw_support">
-        <xacro:default_inertial mass="0.05"/>
+        <xacro:default_inertial mass="0.004"/>
         <visual>
             <origin rpy="0 0 ${PI / 2}" xyz="0 -0.005 -0.015"/>
@@ -94,5 +94,5 @@
     </link>
     <link name="gripper_right">
-        <xacro:default_inertial mass="0.01"/>
+        <xacro:default_inertial mass="0.001"/>
         <visual>
             <origin rpy="0 0 -${PI / 2}" xyz="-0.01 0.050 -0.01"/>
@@ -109,5 +109,5 @@
     </link>
     <link name="gripper_left">
-        <xacro:default_inertial mass="0.01"/>
+        <xacro:default_inertial mass="0.001"/>
         <visual>
             <origin rpy="0 0 -${PI / 2}" xyz="-0.004 0.050 -0.01"/>
