Commit message: initial pca9685 add

File: src/mybots_description/urdf/smallbot_ros2_control.xacro (robot description, xacro)
@@ -33,4 +33,13 @@
             <state_interface name="velocity" />
         </joint>
+    </ros2_control>
+    <ros2_control name="LeftArm" type="system">
+        <!-- ros2_control Real Robot -->
+        <xacro:unless value="$(arg is_sim)">
+            <hardware>
+                <plugin>pca9685_hardware_interface/Pca9685SystemHardware</plugin>
+            </hardware>
+        </xacro:unless>
+        <!-- ros2_control Common Interfaces -->
         <joint name="joint_1">
             <command_interface name="position">
@@ -61,8 +70,4 @@
             <state_interface name="position" />
         </joint>
-        <joint name="joint_5">
-            <param name="mimic">joint_4</param>
-            <param name="multiplier">-1</param>
-        </joint>
     </ros2_control>
 </robot>
