Commit message: bigbot wifi dev for PID constants

File: src/mybots_description/urdf/bigbot_physical.urdf.xacro (robot description, xacro)
@@ -17,5 +17,5 @@
     <inertial>
       <origin xyz="-0.070489 -0.000718 0.040699" rpy="0.0 0.0 0.0" />
-      <mass value="1.409448"/>
+      <mass value="10.0"/>
       <inertia ixx="0.011114" ixy="0.000188" ixz="-0.005821"
                iyy="0.017229" iyz="0.000127"
@@ -39,5 +39,5 @@
     <parent link="base_footprint"/>
     <child link="base_link" />
-    <origin xyz="0 0 0.033" rpy="0 0 0"/>
+    <origin xyz="0 0 0.063" rpy="0 0 0"/>
   </joint>
   <link name="wheel_right_link">
@@ -59,10 +59,10 @@
       <origin xyz="0 -0.015 0" rpy="1.57 0 0" />
       <geometry>
-        <sphere radius="0.033"/>
+        <sphere radius="0.063"/>
       </geometry>
     </collision>
   </link>
   <joint name="wheel_right_joint" type="continuous">
-    <origin xyz="0 -0.141 0" rpy="0 0 0" />
+    <origin xyz="0 -0.2225 0" rpy="0 0 0" />
     <parent link="base_link" />
     <child link="wheel_right_link" />
@@ -88,10 +88,10 @@
       <origin xyz="0 -0.014 0" rpy="-1.57 0 0" />
       <geometry>
-        <sphere radius="0.033"/>
+        <sphere radius="0.063"/>
       </geometry>
     </collision>
   </link>
   <joint name="wheel_left_joint" type="continuous">
-    <origin xyz="0 0.141 0" rpy="0 0 0" />
+    <origin xyz="0 0.2225 0" rpy="0 0 0" />
     <parent link="base_link" />
     <child link="wheel_left_link" />
@@ -121,5 +121,5 @@
   </link>
   <joint name="caster_right_joint" type="fixed">
-    <origin xyz="-0.137 -0.095 .0133" rpy="1.57 0 1.57" />
+    <origin xyz="-0.137 -0.095 -.025" rpy="1.57 0 1.57" />
     <parent link="base_link" />
     <child link="caster_right_link" />
@@ -149,5 +149,5 @@
   </link>
   <joint name="caster_left_joint" type="fixed">
-    <origin xyz="-0.137 0.095 0.0133" rpy="1.57 0 1.57" />
+    <origin xyz="-0.137 0.095 -.025" rpy="1.57 0 1.57" />
     <parent link="base_link" />
     <child link="caster_left_link" />
